File: Design Files/BLUv3/PS4_Main_Schematic_V3.sch (EAGLE design)
At the start: 126 parts, among them CN1 505278-1233, CN2 B2B-ZR-SM4-TF, J2 TC2050-IDC-NL, Q1 mmbt2222, Q3 mmbt2222, U1 XMEGA128A1U, U10 TP4056, U11 TPS63020, U12 TPS630250RNCT, U13 TPS82085SILT8-MICRO_SIP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

Commit message: Cleaned up Schematic
Other:
- note added: "2K -> 580mA 1.66K -> 690mA 1.5K -> 780mA 1.33K -> 900mA 1.2K -> 1000mA"
- note added: "3V3 LDO VReg"
- note added: "Button Breakout"
- note added: "Carbon Contact Connector"
- note added: "Design 1: https://webench.ti.com/appinfo/webench/scripts/SDP.cgi?ID=99B4999514CACA22"
- note added: "Design 2: https://webench.ti.com/appinfo/webench/scripts/SDP.cgi?ID=79A04713E1C51173"
- note added: "Design 3: https://webench.ti.com/appinfo/webench/scripts/SDP.cgi?ID=1AA74D5A1DA9D93F"
- note added: "Design 4: https://webench.ti.com/appinfo/webench/scripts/SDP.cgi?ID=06F25B5DB47F4250"
- note added: "GD25Q32CSIGR"
- note added: "JATG and PDI implemented according to the AVR connector on the ATMEL ICE programmer"
- note added: "Li-ion Charger"
- note added: "NRF24L01+ mini"
- note added: "R1 10K -> 130mA 5K -> 250mA 4K -> 300mA 3K -> 400mA"
- note removed: "+5V AUTO SELECTOR"
- note removed: "DAC"
- note removed: "JATG and PDI implemented according to ATMEL ICE connector"
- note removed: "JTAG"
- note removed: "LEDs"
- note removed: "R11 10K -> 130mA 5K -> 250mA 4K -> 300mA 3K -> 400mA 2K -> 580mA 1.66K -> 690mA 1.5K -> 780mA 1.33K -> 900mA 1.2K -> 1000mA"
- note removed: "https://webench.ti.com/appinfo/webench/scripts/SDP.cgi?ID=06F25B5DB47F4250 Rename to Design 4"
- note removed: "https://webench.ti.com/appinfo/webench/scripts/SDP.cgi?ID=1AA74D5A1DA9D93F Rename to Design 3"
- note removed: "https://webench.ti.com/appinfo/webench/scripts/SDP.cgi?ID=79A04713E1C51173 Rename to Design 2"
- note removed: "https://webench.ti.com/appinfo/webench/scripts/SDP.cgi?ID=99B4999514CACA22 Rename to Design 1"
- moved on the sheet: C1, C10, C11, C12, C13, C14, C15, C16, C17, C18, C19, C2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
